File: raspberry-to-caetla.kicad_pcb (KiCad board)
At the start: 2 copper layers, 65 x 30 mm, 22 parts, among them J2 RASPBERRY_PI, J3 PARALLEL, U1 74LVC1G125, U2 74LVC541AT20, U3 74LVC1G125, U4 74LVC1G125, U5 74LVC1G125, U6 74LVC1G125

Commit message: version 1.1
Parts:
- U2: value 74LVC541AT20 -> 74HCT541
- moved G*** 0.72 mm to (107.2, 66.5)
Connections:
- J3 pad 1: /STROBE -> (no net)
- J3 pad 4: (no net) -> /ERROR
- POWER pad 2: /STROBE -> /ERROR
Routing:
- net /STROBE: track 50.5 -> 0.00 mm
- net /ERROR: track 0.00 -> 43.4 mm
- net (no net): track 0.00 -> 0.78 mm
Other:
- board text added: "Raspi-Caetla interface Jakub Czekański v1.1"
- board text removed: "Raspi-Caetla interface Jakub Czekański v1.0"
