File: raspberry-to-caetla.sch (KiCad schematic (older format))
At the start: 17 parts, among them J1 UART, J2 RASPBERRY_PI, J3 PARALLEL, U1 74LVC1G125, U2 74LVC541AT20, U3 74LVC1G125, U4 74LVC1G125, U5 74LVC1G125, U6 74LVC1G125

Commit message: version 1.1
Parts:
- U2: value 74LVC541AT20 -> 74HCT541
Connections:
- net ERROR: now also JP1.2 (B)
- net STROBE: no longer JP1.2 (B)
Changed lines of the file:
@@
 Title "Raspberry to Caetla interface"
 Date "2019-10-01"
-Rev "v1.0"
+Rev "v1.1"
 Comp ""
 Comment1 ""
@@
 P 5600 2550
 F 0 "U2" H 5600 3531 50  0000 C CNN
-F 1 "74LVC541AT20" H 5600 3440 50  0000 C CNN
+F 1 "74HCT541" H 5600 3440 50  0000 C CNN
 F 2 "Package_SO:Infineon_PG-DSO-20-32" H 5600 2550 50  0001 C CNN
 F 3 "http://www.ti.com/lit/gpn/sn74HCT541" H 5600 2550 50  0001 C CNN
@@
 Wire Wire Line
 	6400 1250 6400 1300
-Wire Wire Line
-	6400 1700 6400 1950
-Wire Wire Line
-	6400 1950 7750 1950
 $Comp
 L power:GND #PWR03
@@
 Wire Wire Line
 	2900 3950 2900 4100
+Wire Wire Line
+	8850 2050 8850 1750
+Wire Wire Line
+	8850 1750 6400 1750
+Wire Wire Line
+	6400 1750 6400 1700
+Wire Wire Line
+	8250 2050 8850 2050
 $EndSCHEMATC
